Commit message: establish gazebo enviroment for Journal experiments

File: franka_description/robots/hand.xacro (robot description, xacro)
@@ -13,5 +13,5 @@
       <visual>
         <geometry>
-          <mesh filename="package://franka_description/meshes/visual/hand.dae"/>
+          <mesh filename="package://franka_description/meshes/visual/hand.dae" />
         </geometry>
       </visual>

File: franka_description/robots/panda_arm.urdf.xacro (robot description, xacro)
@@ -35,4 +35,95 @@
       <child  link="$(arg arm_id)_link0" />
     </joint>
+    <!-- added by jyp on 0525 -->
+    <!-- joint definition -->
+    <joint name="camera_joint" type="fixed">
+      <axis xyz="0 1 0" />
+      <origin xyz="-1.05 0.5 1.5" rpy="3.1415927 1.5707963 2.2"/>
+      <parent link="world"/>
+      <child link="camera_link"/>
+    </joint>
+    <!-- link definition -->
+    <!-- Camera -->
+    <link name="camera_link">
+      <collision>
+        <origin xyz="0 0 0" rpy="0 0 0"/>
+        <geometry>
+          <box size="0.1 0.04 0.04"/>
+        </geometry>
+      </collision>
+      <visual>
+        <origin xyz="0 0 0" rpy="0 0 0"/>
+        <geometry>
+          <box size="0.1 0.04 0.04"/>
+        </geometry>
+        <material name="red"/>
+      </visual>
+      <inertial>
+        <mass value="1e-5" />
+        <origin xyz="0 0 0" rpy="0 0 0"/>
+        <inertia ixx="1e-6" ixy="0" ixz="0" iyy="1e-6" iyz="0" izz="1e-6" />
+      </inertial>
+    </link>
+    <!-- ArUco marker -->
+    <joint name="aruco_joint" type="fixed">
+      <origin xyz="0.06 0.06 0.0" rpy="0.0 0.0 0.785398"/>
+      <parent link="$(arg arm_id)_link8"/>
+      <child link="aruco_link"/>
+    </joint>
+    <link name="aruco_link">
+      <collision>
+        <origin xyz="-0.04 -0.034 0.050" rpy="-1.5707963267949 0 -1.5707963267949"/>
+        <geometry>
+          <box size="0.04 0.0001 0.04"/>
+        </geometry>
+      </collision>
+      <visual>
+        <origin xyz="-0.017 -0.0595 0.050" rpy="-1.5707963267949 0 -1.5707963267949"/>
+        <geometry>
+          <box size="0.04 0.001 0.04"/>
+        </geometry>
+        <pose>0 0 0 1 0 0</pose>
+      </visual>
+    </link>
+    <!-- Marker connecter link -->
+    <!-- <joint name="$_marker_joint" type="fixed">
+        <parent link="world"/>
+        <child link="panda_marker_link"/>
+        <origin xyz="0.06 0.06 0.0" rpy="0.0 0.0 0.785398"/>
+    </joint>
+    <link name="panda_marker_link">
+      <collision>
+        <origin xyz="0 0 0" rpy="0 0 0"/>
+        <geometry>
+          <box size="0.1 0.04 0.04"/>
+        </geometry>
+      </collision>
+      <visual name='visual'>
+        <origin xyz="-0.04 -0.017 0.053" rpy="-1.5707963267949 0 -1.5707963267949"/>
+        <geometry>
+          <mesh filename="package://franka_description/meshes/collision/Franka_connecter.stl" scale="0.001 0.001 0.001" />
+        </geometry>
+        <pose>0 0 0 1 0 0</pose>
+      </visual>
+      <inertial>
+        <mass value="1e-5" />
+        <origin xyz="0 0 0" rpy="0 0 0"/>
+        <inertia ixx="1e-6" ixy="0" ixz="0" iyy="1e-6" iyz="0" izz="1e-6" />
+      </inertial>
+    </link> -->
+    <!-- ArUco marker -->
+    <joint name="marker_joint" type="fixed">
+      <parent link="$(arg arm_id)_link8"/>
+      <child link="marker_link"/>
+      <origin xyz="0.06 0.06 0.0" rpy="0.0 0.0 0.785398"/>
+    </joint>
+    <link name="marker_link">
+      <visual name="visual">
+        <origin xyz="-0.04 -0.016 0.053" rpy="-1.5707963267949 0 -1.5707963267949"/>
+        <geometry>
+          <mesh filename="package://franka_description/meshes/collision/Franka_connecter.stl" scale="0.001 0.001 0.001" />
+        </geometry>
+      </visual>
+    </link>
     <xacro:gazebo-joint joint="$(arg arm_id)_joint1" transmission="hardware_interface/PositionJointInterface" />
     <xacro:gazebo-joint joint="$(arg arm_id)_joint2" transmission="hardware_interface/PositionJointInterface" />

File: franka_description/robots/panda_gazebo.xacro (robot description, xacro)
@@ -356,4 +356,51 @@
       <mimic joint="${arm_id}_finger_joint1" />
     </joint>
+    <!-- added by jyp on 0525 -->
+    <!-- Sensor configuration-->
+    <!-- camera -->
+    <gazebo reference="camera_link">
+      <material>Gazebo/Blue</material>
+      <sensor type="camera" name="camera1">
+        <update_rate>30.0</update_rate>
+        <camera name="head">
+          <horizontal_fov>0.5</horizontal_fov>
+          <image>
+            <width>1920</width>
+            <height>1080</height>
+            <format>R8G8B8</format>
+          </image>
+          <clip>
+            <near>0.02</near>
+            <far>300</far>
+          </clip>
+          <noise>
+            <type>gaussian</type>
+            <!-- Noise is sampled independently per pixel on each frame.
+                 That pixel's noise value is added to each of its color
+                 channels, which at that point lie in the range [0,1]. -->
+            <mean>0.0</mean>
+            <stddev>0.007</stddev>
+          </noise>
+        </camera>
+        <!--gazebo_ros/gazebo_ros_camera.cpp-->
+        <plugin name="camera_controller" filename="libgazebo_ros_camera.so">
+          <alwaysOn>true</alwaysOn>
+          <updateRate>0.0</updateRate>
+          <cameraName>/franka/camera1</cameraName>
+          <imageTopicName>image_raw</imageTopicName>
+          <cameraInfoTopicName>camera_info</cameraInfoTopicName>
+          <frameName>camera_link</frameName>
+          <hackBaseline>0.07</hackBaseline>
+          <distortionK1>0.0</distortionK1>
+          <distortionK2>0.0</distortionK2>
+          <distortionK3>0.0</distortionK3>
+          <distortionT1>0.0</distortionT1>
+          <distortionT2>0.0</distortionT2>
+        </plugin>
+      </sensor>
+    </gazebo>
+    <gazebo reference="aruco_link">
+      <material>Gazebo/aruco-98</material>
+    </gazebo>
   </xacro:macro>
 </robot>
