Commit message: modified gazebo simulator

File: franka_description/robots/panda_arm.urdf.xacro (robot description, xacro)
@@ -57,5 +57,5 @@
           <box size="0.1 0.04 0.04"/>
         </geometry>
-        <material name="red"/>
+        <cast_shadows>false</cast_shadows>
       </visual>
       <inertial>
@@ -84,4 +84,5 @@
         </geometry>
         <pose>0 0 0 1 0 0</pose>
+        <cast_shadows>false</cast_shadows>
       </visual>
     </link>
@@ -124,4 +125,5 @@
           <mesh filename="package://franka_description/meshes/collision/Franka_connecter.stl" scale="0.001 0.001 0.001" />
         </geometry>
+        <cast_shadows>false</cast_shadows>
       </visual>
     </link>

File: franka_description/robots/panda_arm.xacro (robot description, xacro)
@@ -16,4 +16,5 @@
           <mesh filename="package://${description_pkg}/meshes/visual/link0.dae"/>
         </geometry>
+        <cast_shadows>false</cast_shadows>
       </visual>
       <collision>
@@ -41,4 +42,5 @@
           <mesh filename="package://${description_pkg}/meshes/visual/link1.dae"/>
         </geometry>
+        <cast_shadows>false</cast_shadows>
       </visual>
       <collision>
@@ -74,4 +76,5 @@
           <mesh filename="package://${description_pkg}/meshes/visual/link2.dae"/>
         </geometry>
+        <cast_shadows>false</cast_shadows>
       </visual>
       <collision>
@@ -107,4 +110,5 @@
           <mesh filename="package://${description_pkg}/meshes/visual/link3.dae"/>
         </geometry>
+        <cast_shadows>false</cast_shadows>
       </visual>
       <collision>
@@ -140,4 +144,5 @@
           <mesh filename="package://${description_pkg}/meshes/visual/link4.dae"/>
         </geometry>
+        <cast_shadows>false</cast_shadows>
       </visual>
       <collision>
@@ -173,4 +178,5 @@
           <mesh filename="package://${description_pkg}/meshes/visual/link5.dae"/>
         </geometry>
+        <cast_shadows>false</cast_shadows>
       </visual>
       <collision>
@@ -224,4 +230,5 @@
           <mesh filename="package://${description_pkg}/meshes/visual/link6.dae"/>
         </geometry>
+        <cast_shadows>false</cast_shadows>
       </visual>
       <collision>
@@ -257,4 +264,5 @@
           <mesh filename="package://${description_pkg}/meshes/visual/link7.dae"/>
         </geometry>
+        <cast_shadows>false</cast_shadows>
       </visual>
       <collision>

File: franka_description/robots/panda_gazebo.xacro (robot description, xacro)
@@ -24,4 +24,5 @@
           <mesh filename="package://franka_description/meshes/visual/link0.dae"/>
         </geometry>
+        <cast_shadows>false</cast_shadows>
       </visual>
       <collision>
@@ -46,4 +47,5 @@
           <mesh filename="package://franka_description/meshes/visual/link1.dae"/>
         </geometry>
+        <cast_shadows>false</cast_shadows>
       </visual>
       <collision>
@@ -76,4 +78,5 @@
           <mesh filename="package://franka_description/meshes/visual/link2.dae"/>
         </geometry>
+        <cast_shadows>false</cast_shadows>
       </visual>
       <collision>
@@ -106,4 +109,5 @@
           <mesh filename="package://franka_description/meshes/visual/link3.dae"/>
         </geometry>
+        <cast_shadows>false</cast_shadows>
       </visual>
       <collision>
@@ -136,4 +140,5 @@
           <mesh filename="package://franka_description/meshes/visual/link4.dae"/>
         </geometry>
+        <cast_shadows>false</cast_shadows>
       </visual>
       <collision>
@@ -166,4 +171,5 @@
           <mesh filename="package://franka_description/meshes/visual/link5.dae"/>
         </geometry>
+        <cast_shadows>false</cast_shadows>
       </visual>
       <collision>
@@ -196,4 +202,5 @@
           <mesh filename="package://franka_description/meshes/visual/link6.dae"/>
         </geometry>
+        <cast_shadows>false</cast_shadows>
       </visual>
       <collision>
@@ -226,4 +233,5 @@
           <mesh filename="package://franka_description/meshes/visual/link7.dae"/>
         </geometry>
+        <cast_shadows>false</cast_shadows>
       </visual>
       <collision>
@@ -272,4 +280,5 @@
           <mesh filename="package://franka_description/meshes/visual/hand.dae"/>
         </geometry>
+        <cast_shadows>false</cast_shadows>
       </visual>
       <collision>
@@ -322,4 +331,5 @@
           <mesh filename="package://franka_description/meshes/visual/finger.dae"/>
         </geometry>
+        <cast_shadows>false</cast_shadows>
       </visual>
       <xacro:finger-collision sign="+" />
@@ -332,4 +342,5 @@
           <mesh filename="package://franka_description/meshes/visual/finger.dae"/>
         </geometry>
+        <cast_shadows>false</cast_shadows>
       </visual>
       <xacro:finger-collision sign="-" />
@@ -361,4 +372,7 @@
     <gazebo reference="camera_link">
       <material>Gazebo/Blue</material>
+      <visual>
+        <cast_shadows>false</cast_shadows>
+      </visual>
       <sensor type="camera" name="camera1">
         <update_rate>30.0</update_rate>

Commit message: change model.sdf, stone.sdf and panda_arm.urdf.xacro

File: franka_description/robots/panda_arm.urdf.xacro (robot description, xacro)
@@ -39,5 +39,6 @@
     <joint name="camera_joint" type="fixed">
       <axis xyz="0 1 0" />
-      <origin xyz="-1.05 0.5 1.5" rpy="3.1415927 1.5707963 2.2"/>
+      <!-- <origin xyz="-1.05 0.5 1.5" rpy="3.1415927 1.5707963 2.2"/> -->
+      <origin xyz="-0.5 0.5 1.5" rpy="3.1415927 1.5707963 1.57"/>
       <parent link="world"/>
       <child link="camera_link"/>
